File: hardware/rpi_cm4_cm5_CarrierBoard/rpi_cm4_cm5_CarrierBoard.kicad_pcb (KiCad board)
At the start: 8 copper layers, 181.6 x 100.6 mm, 667 parts, among them J1 DM3AT-SF-PEJM5, J10 PR20206VBNN, J11 MIKROE-4247, J12 RPI_CMx_B, J13 SJ-3523-SMT-TR, J14 SJ-3523-SMT-TR, J15 694106301002, J16 12401598E4#2A, J17 5051102291, J19 RPI_CMx_A, J2 0484050003, J21 61300311121, J22 61300311121, J23 MDT420M03001, J24 SM04B-SRSS-TB, J3 0484050003, J4 2086581001, J5 0826-1X1T-32-F, J7 2998TR, J8 62684-402100ALF, J9 5051101092, Q1 DMPH6050SK3-13, Q10 SSM3K56FS,LF, Q11 SSM3K56FS,LF, Q12 2N7002, Q13 2N7002, Q14 2N7002, Q15 2N7002, Q16 DMP3030SN-7, Q18 MMBT3904-7-F, Q19 2N7002, Q2 2N7002, Q20 2N7002, Q21 2N7002, Q22 SSM3K56FS,LF, Q23 SSM3K56FS,LF, Q24 2N7002, Q25 2N7002, Q26 2N7002, Q3 2N7002, Q4 2N7002, Q5 2N7002, Q6 2N7002, Q7 2N7002, Q8 2N7002, Q9 2N7002, U1 PIC32AK1216GC41064-I/M7, U10 TPS54527DDAR, U11 TPS54527DDAR, U12 TPS7A7001DDAR, U13 INA180A2IDBVR, U14 INA180A2IDBVR, U15 SN65DSI84ZXHR, U16 SN74LVC1G125DBVR, U18 AP22913W6-7, U19 SN74LVC1G125DBVR, U20 STWD100NYWY3F, U21 MCP7940NT-I/MS, U22 FSUSB42UMX, U23 AP22913W6-7, U24 MAX16928CGUP, U25 TPS79901DRVR, U26 TPS61169DCKR, U27 AP22913W6-7, U28 INA180A2IDBVR, U3 SE555DR, U30 STM6710DWB6F, U31 SN74LVC1G125DBVR, U32 SN74HCS365QPWRQ1, U33 SGTL5000XNBA3R2, U34 12MHz, U35 SN74HCS365QPWRQ1, U36 INA180A2IDBVR, U37 SN74LVC1G14DBVR, U38 ASAK-32.768KHZ-LRS-T, U4 AP22913W6-7, U6 SST25VF512A, U7 UPD720202K8-711-BAA-A, U8 AP2192AFGEG-7, U9 TPS54527DDAR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

Commit message: design review add new rev of output job files
Routing:
- net /MKB1.~{RST}: track 26.6 -> 22.6 mm, vias 2 -> 1
- net Net-(D32-K): track 33.4 -> 31.0 mm
- net Net-(D31-K): track 32.7 -> 30.3 mm
- net Net-(D33-K): track 32.8 -> 30.6 mm
- net /PIC32AK1216/BTN1: track 59.6 -> 61.2 mm
- net GND: vias 893 -> 890
Other:
- board text added: "Drill file 'rpi_cm4_cm5_CarrierBoard-PTH.drl' contains plated through holes: ============================================================= T1 0.200mm 0.0079{dblquote} (1485 holes) T2 0.200mm 0.0079{dblquote} (30 holes) T3 0.330mm 0.0130{dblquote} (34 holes) T4 0.500mm 0.0197{dblquote} (4 holes) (with 4 slots) T5 0.700mm 0.0276{dblquote} (21 holes) (with 3 slots) T6 0.890mm 0.0350{dblquote} (12 ho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"
- board text removed: "Drill report for rpi_cm4_cm5_CarrierBoard.kicad_pcb Created on 2026-02-15T12:01:54-0500 Drill file 'rpi_cm4_cm5_CarrierBoard-PTH.drl' contains plated through holes: ============================================================= T1 0.200mm 0.0079{dblquote} (1489 holes) T2 0.200mm 0.0079{dblquote} (30 holes) T3 0.330mm 0.0130{dblquote} (34 holes) T4 0.500mm 0.0197{dblquote} (4 holes) (with 4 slots) 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"
