File: hardware/rpi_cm4_cm5_CarrierBoard/Ethernet.kicad_sch (KiCad schematic)
At the start: 11 parts, among them J5 0826-1X1T-32-F

Commit message: Significant update in PCB layout; Completed preliminary high speed rules definition and fanout of differential pairs + GND vias. Started routing high speed signals Slight changes to Pinout based on component placement
Connections:
- net ETH_P0_N: now also D13.4 (I/O3); no longer D13.2 (I/O2)
- net ETH_P0_P: now also D13.5 (I/O4); no longer D13.1 (I/O1)
- net ETH_P1_N: now also D13.2 (I/O2); no longer D13.5 (I/O4)
- net ETH_P1_P: now also D13.1 (I/O1); no longer D13.4 (I/O3)
- net ETH_P2_N: now also D14.7 (I/O5); no longer D13.8 (I/O6)
- net ETH_P2_P: now also D14.8 (I/O6); no longer D13.7 (I/O5)
- net ETH_P3_N: now also D14.5 (I/O4); no longer D14.2 (I/O2)
- net ETH_P3_P: now also D14.4 (I/O3); no longer D14.1 (I/O1)
- net ETH_~{LED1}: now also D13.8 (I/O6); no longer D14.7 (I/O5)
- net ETH_~{LED2}: now also D14.1 (I/O1); no longer D14.4 (I/O3)
- net ETH_~{LED3}: now also D13.7 (I/O5); no longer D14.5 (I/O4)
