File: hardware/rpi_cm4_cm5_CarrierBoard/TFT_CONN.kicad_sch (KiCad schematic)
At the start: 30 parts, among them J8 62684-402100ALF, J9 5051101092

Commit message: Continue working on the layout. Completed most of power planes planning and pouring Completed all DiffPairs routing and length matching (preliminary)
Connections:
- net TFT_LED+ renamed TFT_LEDP
- net TFT_LED- renamed TFT_LEDM
Changed lines of the file:
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@@
 		)
 	)
-	(hierarchical_label "TFT_LED+"
+	(hierarchical_label "TFT_LEDP"
 		(shape input)
 		(at 152.4 130.81 180)
@@
 		)
 	)
-	(hierarchical_label "TFT_LED-"
+	(hierarchical_label "TFT_LEDM"
 		(shape output)
 		(at 152.4 133.35 180)

Commit message: Significant update Stackup changed from 6 to 8 layers Changed design notes accordingly Re-routed all differential pairs and length match / skew match Fanout critical signals away from dense areas 95% routing completed
Parts:
- removed C244: 0.1u, footprint:CAP_NONPOL_0402, symbol KicadCompDb:Capacitors/CAP_CER_SMT_00001
- removed C246: 1u, footprint:CAP_NONPOL_0805, symbol KicadCompDb:Capacitors/CAP_CER_SMT_00002
- removed R291, R293, R294, R295, R296: 0R, footprint:RES_0402, symbol KicadCompDb:Resistors/RES_SMT_00001
- removed R292: 10K, footprint:RES_0402, symbol KicadCompDb:Resistors/RES_SMT_00013
Connections:
- net at J9.4 (I2C_~{RST}): no longer D23.4 (I/O3)
- net at J9.1 (I2C_SDA): no longer D23.8 (I/O6)
- net at J9.2 (I2C_~{INT}): no longer D23.7 (I/O5)
- net at J9.3 (I2C_SCL): no longer D23.5 (I/O4)
- no-connect marks 3 -> 12
Other:
- note removed: "Default = USB touch"
- note removed: "Mix to ease routing"

Commit message: Add preliminary output files (PCB PDF, Gerbers, IPC-D-356, IPC-2581, Pick_N_Place, etc) Update BOM, SCH PDF Commit PCB design and set to "Review" state
Parts:
- MTG5, MTG6, MTG7, MTG8: now not fitted; now in the parts list
Changed lines of the file:
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@@
 	(title_block
 		(title "RPI CMx Carrier")
-		(date "2026-02-13")
+		(date "2026-02-15")
 		(rev "2.00-0A")
 		(comment 1 "Jean-Francois Bilodeau")
@@
 		(comment 6 "Jean-Francois Bilodeau")
 		(comment 7 "Not applicable")
-		(comment 8 "Preliminary")
+		(comment 8 "Released")
 		(comment 9 "RPI_CMx_Carrier_2.00-0A_BOM")
 	)
@@
 		(unit 1)
 		(exclude_from_sim no)
-		(in_bom no)
-		(on_board yes)
-		(dnp no)
+		(in_bom yes)
+		(on_board no)
+		(dnp yes)
 		(property "Reference" "MTG7"
 			(at 124.46 181.229 0)
@@
 		(unit 1)
 		(exclude_from_sim no)
-		(in_bom no)
-		(on_board yes)
-		(dnp no)
+		(in_bom yes)
+		(on_board no)
+		(dnp yes)
 		(property "Reference" "MTG8"
 			(at 130.302 181.356 0)
@@
 		(unit 1)
 		(exclude_from_sim no)
-		(in_bom no)
-		(on_board yes)
-		(dnp no)
+		(in_bom yes)
+		(on_board no)
+		(dnp yes)
 		(property "Reference" "MTG6"
 			(at 130.302 175.641 0)
@@
 		(unit 1)
 		(exclude_from_sim no)
-		(in_bom no)
-		(on_board yes)
-		(dnp no)
+		(in_bom yes)
+		(on_board no)
+		(dnp yes)
 		(property "Reference" "MTG5"
 			(at 124.46 175.641 0)

Commit message: Update BOM build options (DNP, Exclude from board, etc) Export new BOM and new schematic
Parts:
- MTG5, MTG6, MTG7, MTG8: now fitted; now left out of the parts list
Changed lines of the file:
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@@
 		(unit 1)
 		(exclude_from_sim no)
-		(in_bom yes)
-		(on_board no)
-		(dnp yes)
+		(in_bom no)
+		(on_board yes)
+		(dnp no)
 		(property "Reference" "MTG7"
 			(at 124.46 181.229 0)
@@
 		(unit 1)
 		(exclude_from_sim no)
-		(in_bom yes)
-		(on_board no)
-		(dnp yes)
+		(in_bom no)
+		(on_board yes)
+		(dnp no)
 		(property "Reference" "MTG8"
 			(at 130.302 181.356 0)
@@
 		(unit 1)
 		(exclude_from_sim no)
-		(in_bom yes)
-		(on_board no)
-		(dnp yes)
+		(in_bom no)
+		(on_board yes)
+		(dnp no)
 		(property "Reference" "MTG6"
 			(at 130.302 175.641 0)
@@
 		(unit 1)
 		(exclude_from_sim no)
-		(in_bom yes)
-		(on_board no)
-		(dnp yes)
+		(in_bom no)
+		(on_board yes)
+		(dnp no)
 		(property "Reference" "MTG5"
 			(at 124.46 175.641 0)

Commit message: Add test points on relevant signals Re-generate SCH_PDF Re-generate BOM Re-generate all gerbers and relevant PCB output files (still in review phase)
Parts:
- ITEM2: now not fitted
- MTG5, MTG6, MTG7, MTG8: Package (none) -> M2.5; now not fitted
Changed lines of the file:
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@@
 	(title_block
 		(title "RPI CMx Carrier")
-		(date "2026-02-15")
+		(date "2026-02-17")
 		(rev "2.00-0A")
 		(comment 1 "Jean-Francois Bilodeau")
@@
 	(symbol
 		(lib_id "KicadCompDb:Miscellaneous/MISC_00004")
-		(at 125.73 182.245 0)
+		(at 125.73 184.15 0)
 		(unit 1)
 		(exclude_from_sim no)
 		(in_bom no)
-		(on_board yes)
-		(dnp no)
+		(on_board no)
+		(dnp yes)
 		(property "Reference" "MTG7"
-			(at 124.46 181.229 0)
+			(at 124.46 183.134 0)
 			(effects
 				(font
@@
 		)
 		(property "Value" "M0504-25-AL-7"
-			(at 129.54 185.1024 0)
+			(at 129.54 187.0074 0)
 			(effects
 				(font
@@
 		)
 		(property "Footprint" "footprint:M0504-25-AL-7"
-			(at 125.73 182.245 0)
+			(at 125.73 184.15 0)
 			(effects
 				(font
@@
 		)
 		(property "Datasheet" "https://dpk3n3gg92jwt.cloudfront.net/domains/raf/pdf/RAF_catalog_0282.pdf"
-			(at 125.73 182.245 0)
+			(at 125.73 184.15 0)
 			(effects
 				(font
@@
 		)
 		(property "Description" "ROUND SPACER M2.5 ALUMINUM 5MM"
-			(at 125.73 182.245 0)
+			(at 125.73 184.15 0)
 			(effects
 				(font
@@
 		)
 		(property "Type" "ROUND SPACER M2.5 ALUMINUM 5MM"
-			(at 125.73 182.245 0)
+			(at 125.73 184.15 0)
 			(show_name yes)
 			(effects
@@
 		)
 		(property "Operating Temperature" "-40°C ~ 150°C"
-			(at 125.73 182.245 0)
+			(at 125.73 184.15 0)
 			(show_name yes)
 			(effects
@@
 		)
 		(property "Dimensions" "4.50mm x 5.00mm"
-			(at 125.73 182.245 0)
+			(at 125.73 184.15 0)
 			(show_name yes)
 			(effects
@@
 		)
 		(property "Manufacturer" "RAF Electronic Hardware"
-			(at 125.73 182.245 0)
+			(at 125.73 184.15 0)
 			(show_name yes)
 			(effects
@@
 		)
 		(property "Manufacturer Part Number" "M0504-25-AL-7"
-			(at 125.73 182.245 0)
+			(at 125.73 184.15 0)
 			(show_name yes)
 			(effects
@@
 		)
 		(property "Distributor" "DigiKey"
-			(at 125.73 182.245 0)
+			(at 125.73 184.15 0)
 			(show_name yes)
 			(effects
@@
 		)
 		(property "Distributor Part Number" "1772-M0504-25-AL-7-ND"
-			(at 125.73 182.245 0)
+			(at 125.73 184.15 0)
 			(show_name yes)
 			(effects
@@
 			)
 		)
+		(property "Package" "M2.5"
+			(at 125.73 184.15 0)
+			(effects
+				(font
+					(size 1.27 1.27)
+				)
+				(hide yes)
+			)
+		)
 		(instances
 			(project "rpi_cm4_cm5_CarrierBoard"
@@
 		(in_bom no)
 		(on_board yes)
-		(dnp no)
+		(dnp yes)
 		(property "Reference" "ITEM2"
 			(at 146.177 173.736 0)
@@
 	(symbol
 		(lib_id "KicadCompDb:Miscellaneous/MISC_00004")
-		(at 130.81 182.245 0)
+		(at 130.81 184.15 0)
 		(unit 1)
 		(exclude_from_sim no)
 		(in_bom no)
-		(on_board yes)
-		(dnp no)
+		(on_board no)
+		(dnp yes)
 		(property "Reference" "MTG8"
-			(at 130.302 181.356 0)
+			(at 130.302 183.261 0)
 			(effects
 				(font
@@
 		)
 		(property "Value" "M0504-25-AL-7"
-			(at 134.62 185.1024 0)
+			(at 134.62 187.0074 0)
 			(effects
 				(font
@@
 		)
 		(property "Footprint" "footprint:M0504-25-AL-7"
-			(at 130.81 182.245 0)
+			(at 130.81 184.15 0)
 			(effects
 				(font
@@
 		)
 		(property "Datasheet" "https://dpk3n3gg92jwt.cloudfront.net/domains/raf/pdf/RAF_catalog_0282.pdf"
-			(at 130.81 182.245 0)
+			(at 130.81 184.15 0)
 			(effects
 				(font
@@
 		)
 		(property "Description" "ROUND SPACER M2.5 ALUMINUM 5MM"
-			(at 130.81 182.245 0)
+			(at 130.81 184.15 0)
 			(effects
 				(font
@@
 		)
 		(property "Type" "ROUND SPACER M2.5 ALUMINUM 5MM"
-			(at 130.81 182.245 0)
+			(at 130.81 184.15 0)
 			(show_name yes)
 			(effects
@@
 		)
 		(property "Operating Temperature" "-40°C ~ 150°C"
-			(at 130.81 182.245 0)
+			(at 130.81 184.15 0)
 			(show_name yes)
 			(effects
@@
 		)
 		(property "Dimensions" "4.50mm x 5.00mm"
-			(at 130.81 182.245 0)
+			(at 130.81 184.15 0)
 			(show_name yes)
 			(effects
@@
 		)
 		(property "Manufacturer" "RAF Electronic Hardware"
-			(at 130.81 182.245 0)
+			(at 130.81 184.15 0)
 			(show_name yes)
 			(effects
@@
 		)
 		(property "Manufacturer Part Number" "M0504-25-AL-7"
-			(at 130.81 182.245 0)
+			(at 130.81 184.15 0)
 			(show_name yes)
 			(effects
@@
 		)
 		(property "Distributor" "DigiKey"
-			(at 130.81 182.245 0)
+			(at 130.81 184.15 0)
 			(show_name yes)
 			(effects
@@
 		)
 		(property "Distributor Part Number" "1772-M0504-25-AL-7-ND"
-			(at 130.81 182.245 0)
+			(at 130.81 184.15 0)
 			(show_name yes)
 			(effects
@@
 			)
 		)
+		(property "Package" "M2.5"
+			(at 130.81 184.15 0)
+			(effects
+				(font
+					(size 1.27 1.27)
+				)
+				(hide yes)
+			)
+		)
 		(instances
 			(project "rpi_cm4_cm5_CarrierBoard"
@@
 		(exclude_from_sim no)
 		(in_bom no)
-		(on_board yes)
-		(dnp no)
+		(on_board no)
+		(dnp yes)
 		(property "Reference" "MTG6"
 			(at 130.302 175.641 0)
@@
 			)
 		)
+		(property "Package" "M2.5"
+			(at 130.81 176.53 0)
+			(effects
+				(font
+					(size 1.27 1.27)
+				)
+				(hide yes)
+			)
+		)
 		(instances
 			(project "rpi_cm4_cm5_CarrierBoard"
@@
 		(exclude_from_sim no)
 		(in_bom no)
-		(on_board yes)
-		(dnp no)
+		(on_board no)
+		(dnp yes)
 		(property "Reference" "MTG5"
 			(at 124.46 175.641 0)
@@
 			(effects
 				(font
+					(size 1.27 1.27)
+				)
+				(hide yes)
+			)
+		)
+		(property "Package" "M2.5"
+			(at 125.73 176.53 0)
+			(effects
+				(font
