File: hardware/rpi_cm4_cm5_CarrierBoard/M2_Expansion.kicad_sch (KiCad schematic)
At the start: 20 parts, among them J23 MDT420M03001, U38 ASAK-32.768KHZ-LRS-T

Commit message: Update schematic sheets (assembly variants, default cap / res notes)
Other:
- note added: "Resistors are 1% 1/16W 0402 unless otherwise noted Capacitors are 10% 50V X7R 0402 unless otherwise noted"
Changed lines of the file:
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@@
 	(title_block
 		(title "RPI CMx Carrier")
-		(date "2026-02-20")
+		(date "2026-02-22")
 		(rev "2.00-0A")
 		(comment 1 "Jean-Francois Bilodeau")
@@
 		(comment 9 "RPI_CMx_Carrier_2.00-0A_BOM")
 	)
+	(text "Resistors are 1% 1/16W 0402 unless otherwise noted\nCapacitors are 10% 50V X7R 0402 unless otherwise noted"
+		(exclude_from_sim no)
+		(at 12.7 170.688 0)
+		(effects
+			(font
+				(size 1.27 1.27)
+			)
+			(justify left)
+		)
+	)
 	(junction

Commit message: Update 12MHz oscillator on Audio Codec schematic sheet to solve single source issue and uncommon packaging. Re-generate all output files including schematics and BOM, as well as all PCB output files
Changed lines of the file:
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@@
 	(title_block
 		(title "RPI CMx Carrier")
-		(date "2026-02-22")
+		(date "2026-02-24")
 		(rev "2.00-0A")
 		(comment 1 "Jean-Francois Bilodeau")
