File: hardware/rpi_cm4_cm5_CarrierBoard/rpi_cm4_cm5_CarrierBoard.kicad_sch (KiCad schematic)
At the start: 22 parts, among them J21 61300311121, J22 61300311121, J24 SM04B-SRSS-TB, U37 SN74LVC1G14DBVR

Commit message: Update BOM build options (DNP, Exclude from board, etc) Export new BOM and new schematic
Parts:
- FID1, FID2, FID3, FID4, FID5, FID6: now left out of the parts list
Changed lines of the file:
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@@
 		(unit 1)
 		(exclude_from_sim no)
-		(in_bom yes)
+		(in_bom no)
 		(on_board yes)
 		(dnp no)
@@
 		(unit 1)
 		(exclude_from_sim no)
-		(in_bom yes)
+		(in_bom no)
 		(on_board yes)
 		(dnp no)
@@
 		(unit 1)
 		(exclude_from_sim no)
-		(in_bom yes)
+		(in_bom no)
 		(on_board yes)
 		(dnp no)
@@
 		(unit 1)
 		(exclude_from_sim no)
-		(in_bom yes)
+		(in_bom no)
 		(on_board yes)
 		(dnp no)
@@
 		(unit 1)
 		(exclude_from_sim no)
-		(in_bom yes)
+		(in_bom no)
 		(on_board yes)
 		(dnp no)
@@
 		(unit 1)
 		(exclude_from_sim no)
-		(in_bom yes)
+		(in_bom no)
 		(on_board yes)
 		(dnp no)

Commit message: Add test points on relevant signals Re-generate SCH_PDF Re-generate BOM Re-generate all gerbers and relevant PCB output files (still in review phase)
Parts:
- added TP10, TP9: 28 mils, footprint:SMT_TP_28_MILS, symbol KicadCompDb:Test Point/TP_00001
- FID1, FID2, FID3, FID4, FID5, FID6: now not fitted
Connections:
- net I2C6.I2C_SCL: now also TP9.1
- net I2C6.I2C_SDA: now also TP10.1

Commit message: Clear ERC markers and cleaned unconnected nets Design freeze
Other:
- sheet RESET_SUPERVISOR ports: added none; removed EXP_IO_~{RST}
Changed lines of the file:
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@@
 	(title_block
 		(title "RPI CMx Carrier")
-		(date "2026-02-26")
+		(date "2026-02-28")
 		(rev "2.00-0A")
 		(comment 1 "Jean-Francois Bilodeau")
@@
 	(wire
 		(pts
-			(xy 182.88 92.075) (xy 198.755 92.075)
-		)
-		(stroke
-			(width 0)
-			(type default)
-		)
-	)
-	(wire
-		(pts
 			(xy 38.735 138.43) (xy 31.115 138.43)
 		)
@@
 		)
 	)
-	(label "EXP_IO_~{RST}"
-		(at 198.755 92.075 180)
-		(effects
-			(font
-				(size 1.27 1.27)
-			)
-			(justify right bottom)
-		)
-	)
 	(label "USB_HUB_~{RST}"
 		(at 61.595 52.705 180)
@@
 			(effects
 				(font
-					(size 1.27 1.27)
-				)
-				(justify right)
-			)
-		)
-		(pin "EXP_IO_~{RST}" output
-			(at 182.88 92.075 0)
-			(effects
-				(font
